File: deska.sch (EAGLE design)
At the start: 10 parts

Commit message: +
Parts:
- added R2: 220, rcl:R-EU_0207/10
- R1: value (none) -> 4k7
Connections:
- removed net N$11: DS18B20-3.KL, R1.1, WEMOS1.3V3
- new net N$12: LED-1.KL, R2.2
- net +5V: now also DS18B20-3.KL, LED-2.KL, R1.1
- net GND: no longer LED-2.KL
- net N$6: now also R2.1; no longer LED-1.KL
Changed lines of the file:
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@@
 <?xml version="1.0" encoding="utf-8"?>
 <!DOCTYPE eagle SYSTEM "eagle.dtd">
-<eagle version="7.7.0">
+<eagle version="9.1.3">
 <drawing>
 <settings>
 <setting alwaysvectorfont="no"/>
+<setting keepoldvectorfont="yes"/>
 <setting verticaltext="up"/>
 </settings>
@@
 <part name="GND1" library="supply1" deviceset="GND" device=""/>
 <part name="GND2" library="supply1" deviceset="GND" device=""/>
-<part name="GND3" library="supply1" deviceset="GND" device=""/>
 <part name="GND5" library="supply1" deviceset="GND" device=""/>
 <part name="GND6" library="supply1" deviceset="GND" device=""/>
@@
 <part name="GND4" library="supply1" deviceset="GND" device=""/>
 <part name="P+3" library="supply1" deviceset="+5V" device=""/>
-<part name="R1" library="rcl" deviceset="R-EU_" device="0207/10"/>
+<part name="R1" library="rcl" deviceset="R-EU_" device="0207/10" value="4k7"/>
 <part name="GND9" library="supply1" deviceset="GND" device=""/>
 <part name="P+4" library="supply1" deviceset="+5V" device=""/>
+<part name="R2" library="rcl" deviceset="R-EU_" device="0207/10" value="220"/>
+<part name="P+5" library="supply1" deviceset="+5V" device=""/>
 </parts>
 <sheets>
@@
 <instance part="GND1" gate="1" x="27.94" y="-7.62"/>
 <instance part="GND2" gate="1" x="27.94" y="27.94"/>
-<instance part="GND3" gate="1" x="27.94" y="20.32"/>
 <instance part="GND5" gate="1" x="27.94" y="58.42"/>
 <instance part="GND6" gate="1" x="27.94" y="68.58"/>
@@
 <instance part="R1" gate="G$1" x="35.56" y="43.18" rot="R90"/>
 <instance part="GND9" gate="1" x="27.94" y="7.62"/>
-<instance part="P+4" gate="1" x="30.48" y="15.24" rot="R270"/>
+<instance part="P+4" gate="1" x="33.02" y="15.24" rot="R270"/>
+<instance part="R2" gate="G$1" x="53.34" y="25.4" rot="R180"/>
+<instance part="P+5" gate="1" x="30.48" y="22.86" rot="R270"/>
 </instances>
 <busses>
@@
 </segment>
 <segment>
-<pinref part="LED" gate="-2" pin="KL"/>
-<pinref part="GND3" gate="1" pin="GND"/>
-</segment>
-<segment>
 <pinref part="RELAY2" gate="-2" pin="KL"/>
 <pinref part="GND5" gate="1" pin="GND"/>
@@
 <net name="N$6" class="0">
 <segment>
-<pinref part="LED" gate="-1" pin="KL"/>
-<wire x1="27.94" y1="25.4" x2="86.36" y2="25.4" width="0.1524" layer="91"/>
+<wire x1="58.42" y1="25.4" x2="86.36" y2="25.4" width="0.1524" layer="91"/>
 <wire x1="86.36" y1="25.4" x2="86.36" y2="48.26" width="0.1524" layer="91"/>
 <pinref part="WEMOS1" gate="D1" pin="D4"/>
 <wire x1="86.36" y1="48.26" x2="78.74" y2="48.26" width="0.1524" layer="91"/>
+<pinref part="R2" gate="G$1" pin="1"/>
 </segment>
 </net>
@@
 <pinref part="PIR" gate="-1" pin="KL"/>
 <pinref part="P+2" gate="1" pin="+5V"/>
+<pinref part="R1" gate="G$1" pin="1"/>
+<wire x1="35.56" y1="38.1" x2="27.94" y2="38.1" width="0.1524" layer="91"/>
+<wire x1="27.94" y1="38.1" x2="27.94" y2="35.56" width="0.1524" layer="91"/>
+<junction x="27.94" y="35.56"/>
+<pinref part="DS18B20" gate="-3" pin="KL"/>
+<wire x1="27.94" y1="45.72" x2="27.94" y2="38.1" width="0.1524" layer="91"/>
+<junction x="27.94" y="38.1"/>
 </segment>
 <segment>
@@
 </segment>
 <segment>
+<pinref part="LED" gate="-2" pin="KL"/>
+<pinref part="P+5" gate="1" pin="+5V"/>
+</segment>
+<segment>
 <pinref part="FLOW" gate="-1" pin="KL"/>
 <pinref part="P+4" gate="1" pin="+5V"/>
+<wire x1="30.48" y1="15.24" x2="27.94" y2="15.24" width="0.1524" layer="91"/>
 </segment>
 </net>
@@
 <net name="N$10" class="0">
 <segment>
+<pinref part="WEMOS1" gate="D1" pin="D8"/>
+<wire x1="38.1" y1="12.7" x2="38.1" y2="45.72" width="0.1524" layer="91"/>
+<wire x1="38.1" y1="45.72" x2="45.72" y2="45.72" width="0.1524" layer="91"/>
 <pinref part="FLOW" gate="-2" pin="KL"/>
 <wire x1="27.94" y1="12.7" x2="38.1" y2="12.7" width="0.1524" layer="91"/>
-<wire x1="38.1" y1="12.7" x2="38.1" y2="45.72" width="0.1524" layer="91"/>
-<pinref part="WEMOS1" gate="D1" pin="D8"/>
-<wire x1="38.1" y1="45.72" x2="45.72" y2="45.72" width="0.1524" layer="91"/>
-</segment>
-</net>
-<net name="N$11" class="0">
-<segment>
-<pinref part="WEMOS1" gate="D1" pin="3V3"/>
-<wire x1="45.72" y1="43.18" x2="40.64" y2="43.18" width="0.1524" layer="91"/>
-<pinref part="DS18B20" gate="-3" pin="KL"/>
-<wire x1="40.64" y1="43.18" x2="33.02" y2="43.18" width="0.1524" layer="91"/>
-<wire x1="27.94" y1="45.72" x2="33.02" y2="45.72" width="0.1524" layer="91"/>
-<wire x1="33.02" y1="45.72" x2="33.02" y2="43.18" width="0.1524" layer="91"/>
-<pinref part="R1" gate="G$1" pin="1"/>
-<wire x1="35.56" y1="38.1" x2="40.64" y2="38.1" width="0.1524" layer="91"/>
-<wire x1="40.64" y1="38.1" x2="40.64" y2="43.18" width="0.1524" layer="91"/>
-<junction x="40.64" y="43.18"/>
-</segment>
-</net>
+</segment>
+</net>
+<net name="N$12" class="0">
+<segment>
+<pinref part="R2" gate="G$1" pin="2"/>
+<pinref part="LED" gate="-1" pin="KL"/>
+<wire x1="27.94" y1="25.4" x2="48.26" y2="25.4" width="0.1524" layer="91"/>
+</segment>
+</net>

Commit message: +
Connections:
- net N$10: now also WEMOS1.D6; no longer WEMOS1.D8
- net N$5: now also WEMOS1.D0; no longer WEMOS1.D3
- net N$7: now also WEMOS1.D3; no longer WEMOS1.D5
- net N$8: now also WEMOS1.D8; no longer WEMOS1.D6

Commit message: board editing
Parts:
- removed I2C: (no value), con-wago-508:W237-04P
- added R3: 220, rcl:R-EU_0207/10
- added SL1: (no value), con-amp-quick:M04
- PIR, SERIAL: device con-wago-508:W237-03P -> con-amp-quick:M03
Connections:
- net +5V: now also PIR.3, SL1.2; no longer I2C-3.KL, PIR-1.KL
- net GND: now also PIR.1, R3.1, SERIAL.1, SL1.1; no longer I2C-4.KL, PIR-3.KL, SERIAL-3.KL
- net N$1: now also SERIAL.2; no longer SERIAL-2.KL
- net N$10: now also R3.2
- net N$2: now also SERIAL.3; no longer SERIAL-1.KL
- net N$3: now also SL1.4; no longer I2C-1.KL
- net N$4: now also SL1.3; no longer I2C-2.KL
- net N$5: now also PIR.2; no longer PIR-2.KL
Changed lines of the file:
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@@
 <?xml version="1.0" encoding="utf-8"?>
 <!DOCTYPE eagle SYSTEM "eagle.dtd">
-<eagle version="9.2.2">
+<eagle version="9.1.3">
 <drawing>
 <settings>
@@
 <part name="RELAY1" library="con-wago-508" deviceset="W237-02P" device=""/>
 <part name="DS18B20" library="con-wago-508" deviceset="W237-03P" device=""/>
-<part name="PIR" library="con-wago-508" deviceset="W237-03P" device=""/>
 <part name="FLOW" library="con-wago-508" deviceset="W237-03P" device=""/>
-<part name="I2C" library="con-wago-508" deviceset="W237-04P" device=""/>
 <part name="RELAY2" library="con-wago-508" deviceset="W237-02P" device=""/>
-<part name="SERIAL" library="con-wago-508" deviceset="W237-03P" device=""/>
 <part name="LED" library="con-wago-508" deviceset="W237-02P" device=""/>
 <part name="WEMOS1" library="esp8266modules" deviceset="WEMOS-D1-MINI" device=""/>
@@
 <part name="R2" library="rcl" deviceset="R-EU_" device="0207/10" value="220"/>
 <part name="P+5" library="supply1" deviceset="+5V" device=""/>
+<part name="PIR" library="con-amp-quick" library_urn="urn:adsk.eagle:library:125" deviceset="M03" device="" package3d_urn="urn:adsk.eagle:package:5957/1"/>
+<part name="SERIAL" library="con-amp-quick" library_urn="urn:adsk.eagle:library:125" deviceset="M03" device="" package3d_urn="urn:adsk.eagle:package:5957/1"/>
+<part name="SL1" library="con-amp-quick" library_urn="urn:adsk.eagle:library:125" deviceset="M04" device="" package3d_urn="urn:adsk.eagle:package:5958/1"/>
+<part name="R3" library="rcl" deviceset="R-EU_" device="0207/10" value="220"/>
 </parts>
 <sheets>
@@
 <attribute name="NAME" x="21.59" y="46.609" size="1.778" layer="95" rot="R180"/>
 </instance>
-<instance part="PIR" gate="-1" x="22.86" y="35.56" smashed="yes">
-<attribute name="NAME" x="21.59" y="36.449" size="1.778" layer="95" rot="R180"/>
-</instance>
-<instance part="PIR" gate="-2" x="22.86" y="33.02" smashed="yes">
-<attribute name="NAME" x="21.59" y="33.909" size="1.778" layer="95" rot="R180"/>
-</instance>
-<instance part="PIR" gate="-3" x="22.86" y="30.48" smashed="yes">
-<attribute name="VALUE" x="22.86" y="33.02" size="1.778" layer="96"/>
-<attribute name="NAME" x="21.59" y="31.369" size="1.778" layer="95" rot="R180"/>
-</instance>
 <instance part="FLOW" gate="-1" x="22.86" y="15.24" smashed="yes">
 <attribute name="NAME" x="21.59" y="16.129" size="1.778" layer="95" rot="R180"/>
@@
 <attribute name="NAME" x="21.59" y="11.049" size="1.778" layer="95" rot="R180"/>
 </instance>
-<instance part="I2C" gate="-1" x="22.86" y="91.44" smashed="yes">
-<attribute name="NAME" x="21.59" y="92.329" size="1.778" layer="95" rot="R180"/>
-</instance>
-<instance part="I2C" gate="-2" x="22.86" y="88.9" smashed="yes">
-<attribute name="NAME" x="21.59" y="89.789" size="1.778" layer="95" rot="R180"/>
-</instance>
-<instance part="I2C" gate="-3" x="22.86" y="86.36" smashed="yes">
-<attribute name="NAME" x="21.59" y="87.249" size="1.778" layer="95" rot="R180"/>
-</instance>
-<instance part="I2C" gate="-4" x="22.86" y="83.82" smashed="yes">
-<attribute name="VALUE" x="22.86" y="86.36" size="1.778" layer="96"/>
-<attribute name="NAME" x="21.59" y="84.709" size="1.778" layer="95" rot="R180"/>
-</instance>
 <instance part="RELAY2" gate="-1" x="22.86" y="63.5" smashed="yes">
 <attribute name="NAME" x="21.59" y="64.389" size="1.778" layer="95" rot="R180"/>
@@
 <attribute name="NAME" x="21.59" y="61.849" size="1.778" layer="95" rot="R180"/>
 </instance>
-<instance part="SERIAL" gate="-1" x="22.86" y="0" smashed="yes">
-<attribute name="NAME" x="21.59" y="0.889" size="1.778" layer="95" rot="R180"/>
-</instance>
-<instance part="SERIAL" gate="-2" x="22.86" y="-2.54" smashed="yes">
-<attribute name="NAME" x="21.59" y="-1.651" size="1.778" layer="95" rot="R180"/>
-</instance>
-<instance part="SERIAL" gate="-3" x="22.86" y="-5.08" smashed="yes">
-<attribute name="VALUE" x="22.86" y="-2.54" size="1.778" layer="96"/>
-<attribute name="NAME" x="21.59" y="-4.191" size="1.778" layer="95" rot="R180"/>
-</instance>
 <instance part="LED" gate="-1" x="22.86" y="25.4" smashed="yes">
 <attribute name="NAME" x="21.59" y="26.289" size="1.778" layer="95" rot="R180"/>
@@
 <instance part="P+5" gate="1" x="30.48" y="22.86" smashed="yes" rot="R270">
 <attribute name="VALUE" x="25.4" y="25.4" size="1.778" layer="96"/>
+</instance>
+<instance part="PIR" gate="G$1" x="20.32" y="33.02"/>
+<instance part="SERIAL" gate="G$1" x="20.32" y="-2.54"/>
+<instance part="SL1" gate="G$1" x="22.86" y="86.36"/>
+<instance part="R3" gate="G$1" x="45.72" y="12.7" smashed="yes" rot="R180">
+<attribute name="NAME" x="49.53" y="11.2014" size="1.778" layer="95" rot="R180"/>
+<attribute name="VALUE" x="49.53" y="16.002" size="1.778" layer="96" rot="R180"/>
 </instance>
 </instances>
@@
 <pinref part="WEMOS1" gate="D1" pin="TX"/>
 <wire x1="93.98" y1="60.96" x2="78.74" y2="60.96" width="0.1524" layer="91"/>
-<pinref part="SERIAL" gate="-2" pin="KL"/>
 <wire x1="27.94" y1="-2.54" x2="93.98" y2="-2.54" width="0.1524" layer="91"/>
+<pinref part="SERIAL" gate="G$1" pin="2"/>
 </segment>
 </net>
@@
 <wire x1="78.74" y1="58.42" x2="91.44" y2="58.42" width="0.1524" layer="91"/>
 <wire x1="91.44" y1="58.42" x2="91.44" y2="0" width="0.1524" layer="91"/>
-<pinref part="SERIAL" gate="-1" pin="KL"/>
 <wire x1="27.94" y1="0" x2="91.44" y2="0" width="0.1524" layer="91"/>
+<pinref part="SERIAL" gate="G$1" pin="3"/>
 </segment>
 </net>
 <net name="GND" class="0">
-<segment>
-<pinref part="SERIAL" gate="-3" pin="KL"/>
-<pinref part="GND1" gate="1" pin="GND"/>
-</segment>
-<segment>
-<pinref part="PIR" gate="-3" pin="KL"/>
-<pinref part="GND2" gate="1" pin="GND"/>
-</segment>
 <segment>
 <pinref part="RELAY2" gate="-2" pin="KL"/>
@@
 <pinref part="RELAY1" gate="-2" pin="KL"/>
 <pinref part="GND6" gate="1" pin="GND"/>
-</segment>
-<segment>
-<pinref part="I2C" gate="-4" pin="KL"/>
-<pinref part="GND7" gate="1" pin="GND"/>
 </segment>
 <segment>
@@
 <pinref part="FLOW" gate="-3" pin="KL"/>
 <pinref part="GND9" gate="1" pin="GND"/>
+<pinref part="R3" gate="G$1" pin="1"/>
+<wire x1="27.94" y1="10.16" x2="50.8" y2="10.16" width="0.1524" layer="91"/>
+<wire x1="50.8" y1="10.16" x2="50.8" y2="12.7" width="0.1524" layer="91"/>
+<junction x="27.94" y="10.16"/>
+</segment>
+<segment>
+<pinref part="GND2" gate="1" pin="GND"/>
+<pinref part="PIR" gate="G$1" pin="1"/>
+</segment>
+<segment>
+<pinref part="GND1" gate="1" pin="GND"/>
+<pinref part="SERIAL" gate="G$1" pin="1"/>
+</segment>
+<segment>
+<pinref part="GND7" gate="1" pin="GND"/>
+<pinref part="SL1" gate="G$1" pin="1"/>
 </segment>
 </net>
 <net name="N$3" class="0">
 <segment>
-<pinref part="I2C" gate="-1" pin="KL"/>
 <wire x1="27.94" y1="91.44" x2="88.9" y2="91.44" width="0.1524" layer="91"/>
 <wire x1="88.9" y1="91.44" x2="88.9" y2="55.88" width="0.1524" layer="91"/>
 <pinref part="WEMOS1" gate="D1" pin="D1"/>
 <wire x1="88.9" y1="55.88" x2="78.74" y2="55.88" width="0.1524" layer="91"/>
+<pinref part="SL1" gate="G$1" pin="4"/>
 </segment>
 </net>
@@
 <wire x1="78.74" y1="53.34" x2="86.36" y2="53.34" width="0.1524" layer="91"/>
 <wire x1="86.36" y1="53.34" x2="86.36" y2="88.9" width="0.1524" layer="91"/>
-<pinref part="I2C" gate="-2" pin="KL"/>
 <wire x1="86.36" y1="88.9" x2="27.94" y2="88.9" width="0.1524" layer="91"/>
+<pinref part="SL1" gate="G$1" pin="3"/>
 </segment>
 </net>
 <net name="N$5" class="0">
 <segment>
-<pinref part="PIR" gate="-2" pin="KL"/>
 <wire x1="43.18" y1="33.02" x2="27.94" y2="33.02" width="0.1524" layer="91"/>
 <pinref part="WEMOS1" gate="D1" pin="D0"/>
 <wire x1="45.72" y1="55.88" x2="43.18" y2="55.88" width="0.1524" layer="91"/>
 <wire x1="43.18" y1="33.02" x2="43.18" y2="55.88" width="0.1524" layer="91"/>
+<pinref part="PIR" gate="G$1" pin="2"/>
 </segment>
 </net>
@@
 </segment>
 <segment>
-<pinref part="PIR" gate="-1" pin="KL"/>
 <pinref part="P+2" gate="1" pin="+5V"/>
 <pinref part="R1" gate="G$1" pin="1"/>
 <wire x1="35.56" y1="38.1" x2="27.94" y2="38.1" width="0.1524" layer="91"/>
 <wire x1="27.94" y1="38.1" x2="27.94" y2="35.56" width="0.1524" layer="91"/>
-<junction x="27.94" y="35.56"/>
 <pinref part="DS18B20" gate="-3" pin="KL"/>
 <wire x1="27.94" y1="45.72" x2="27.94" y2="38.1" width="0.1524" layer="91"/>
 <junction x="27.94" y="38.1"/>
-</segment>
-<segment>
-<pinref part="I2C" gate="-3" pin="KL"/>
+<pinref part="PIR" gate="G$1" pin="3"/>
+<junction x="27.94" y="35.56"/>
+</segment>
+<segment>
 <wire x1="27.94" y1="86.36" x2="33.02" y2="86.36" width="0.1524" layer="91"/>
 <pinref part="P+3" gate="1" pin="+5V"/>
+<pinref part="SL1" gate="G$1" pin="2"/>
 </segment>
 <segment>
@@
 <wire x1="45.72" y1="50.8" x2="40.64" y2="50.8" width="0.1524" layer="91"/>
 <wire x1="40.64" y1="50.8" x2="40.64" y2="12.7" width="0.1524" layer="91"/>
+<pinref part="R3" gate="G$1" pin="2"/>
+<junction x="40.64" y="12.7"/>
 </segment>
 </net>
@@
 which will not be processed correctly with this version.
 </note>
+<note version="8.2" severity="warning">
+Since Version 8.2, EAGLE supports online libraries. The ids
+of those online libraries will not be understood (or retained)
+with this version.
+</note>
+<note version="8.3" severity="warning">
+Since Version 8.3, EAGLE supports URNs for individual library
+assets (packages, symbols, and devices). The URNs of those assets
+will not be understood (or retained) with this version.
+</note>
+<note version="8.3" severity="warning">
+Since Version 8.3, EAGLE supports the association of 3D packages
+with devices in libraries, schematics, and board files. Those 3D
+packages will not be understood (or retained) with this version.
+</note>
 </compatibility>
