File: deska_uprava.brd (EAGLE design)
At the start: 64.4 x 69.8 mm, 11 parts

Commit message: +
Parts:
- added SOURCE: (no value), con-wago-508:W237-132
- RELAYS: device con-amp-quick:04P -> con-wago-508:W237-132
- moved FLOW 1.27 mm to (45.7, 10.2)
- moved LED 1.27 mm to (45.7, 22.9)
- moved RELAYS 1.27 mm to (6.35, 21.6), turned to 270 degrees
Connections:
- net +5V: now also SOURCE.1; no longer RELAYS.2
- net GND: now also SOURCE.2; no longer RELAYS.1
- net N$7: now also RELAYS.1; no longer RELAYS.4
- net N$8: now also RELAYS.2; no longer RELAYS.3
Routing:
- net GND: track 157.8 -> 199.1 mm
- net +5V: track 207.0 -> 175.8 mm
- net N$8: track 10.5 -> 14.3 mm
- net N$7: track 14.8 -> 16.5 mm
- net N$12: track 14.6 -> 13.3 mm
- net N$10: track 55.2 -> 54.0 mm
